Commit message: 20251226

File: kuka_kr210_moveit2/config/kr210_ros2_control.xacro (robot description, xacro)
@@ -1,6 +1,6 @@
 <robot xmlns:xacro="http://www.ros.org/wiki/xacro">
-    <xacro:macro name="kr210_arm_ros2_control" params="name initial_positions_file rsi_config_file">
-        <xacro:property name="initial_positions" value="${load_yaml(initial_positions_file)['initial_positions']}"/>
-        <xacro:property name="rsi_config" value="${load_yaml(rsi_config_file)['rsi']}"/>
+    <xacro:macro name="kr210_arm_ros2_control" params="name position_config_file kuka_rsi_config">
+        <xacro:property name="position_config" value="${load_yaml(position_config_file)['default_position']}"/>
+        <xacro:property name="rsi_config" value="${load_yaml(kuka_rsi_config)['rsi']}"/>
         <ros2_control name="${name}" type="system">
             <hardware>
@@ -20,5 +20,5 @@
                 <command_interface name="position"/>
                 <state_interface name="position">
-                  <param name="initial_value">${initial_positions['joint_1']}</param>
+                  <param name="initial_value">${position_config['joint_1']}</param>
                 </state_interface>
                 <state_interface name="velocity"/>
@@ -27,5 +27,5 @@
                 <command_interface name="position"/>
                 <state_interface name="position">
-                  <param name="initial_value">${initial_positions['joint_2']}</param>
+                  <param name="initial_value">${position_config['joint_2']}</param>
                 </state_interface>
                 <state_interface name="velocity"/>
@@ -34,5 +34,5 @@
                 <command_interface name="position"/>
                 <state_interface name="position">
-                  <param name="initial_value">${initial_positions['joint_3']}</param>
+                  <param name="initial_value">${position_config['joint_3']}</param>
                 </state_interface>
                 <state_interface name="velocity"/>
@@ -41,5 +41,5 @@
                 <command_interface name="position"/>
                 <state_interface name="position">
-                  <param name="initial_value">${initial_positions['joint_4']}</param>
+                  <param name="initial_value">${position_config['joint_4']}</param>
                 </state_interface>
                 <state_interface name="velocity"/>
@@ -48,5 +48,5 @@
                 <command_interface name="position"/>
                 <state_interface name="position">
-                  <param name="initial_value">${initial_positions['joint_5']}</param>
+                  <param name="initial_value">${position_config['joint_5']}</param>
                 </state_interface>
                 <state_interface name="velocity"/>
@@ -55,5 +55,5 @@
                 <command_interface name="position"/>
                 <state_interface name="position">
-                  <param name="initial_value">${initial_positions['joint_6']}</param>
+                  <param name="initial_value">${position_config['joint_6']}</param>
                 </state_interface>
                 <state_interface name="velocity"/>
@@ -62,5 +62,5 @@
                 <command_interface name="position"/>
                 <state_interface name="position">
-                  <param name="initial_value">${initial_positions['left_gripper_finger_joint']}</param>
+                  <param name="initial_value">${position_config['left_gripper_finger_joint']}</param>
                 </state_interface>
                 <state_interface name="velocity"/>
@@ -69,5 +69,5 @@
                 <command_interface name="position"/>
                 <state_interface name="position">
-                  <param name="initial_value">${initial_positions['right_gripper_finger_joint']}</param>
+                  <param name="initial_value">${position_config['right_gripper_finger_joint']}</param>
                 </state_interface>
                 <state_interface name="velocity"/>
